File: HW/Breakout_FDC1004/Breakout_FDC1004.kicad_sch (KiCad schematic)
At the start: 14 parts, among them J1 Conn_Qwiic, J3 Conn_CIN2, J4 Conn_Breadboard, U1 FDC1004

Commit message: Updated BOMs
No PCB changes, just adding Part Number attributes and exporting a table.

Does sneak in a corrected XTAL footprint, but it's not actually applied yet.
Parts:
- C1: value 1u -> 1uF; Manufacturer Part Number (none) -> CL10A105KP8NNNC
- C2: value 0.1u -> 0.1uF; Manufacturer Part Number (none) -> GRM155R61A104KA01J
- D1: Manufacturer Part Number (none) -> 150060GS75000
- J1: Manufacturer Part Number (none) -> SM04B-SRSS-TB
- R1: value 4.7k -> 100Ω; Manufacturer Part Number (none) -> RC0603FR-07100RL
- R2, R3: value 10k -> 10kΩ; Digikey Part Number 311-10.0KHRCT-ND -> (none); Manufacturer Part Number (none) -> RC0603FR-0710KL
- U1: Manufacturer Part Number (none) -> FDC1004DSCR
