File: HW/Breakout_NEH7100_Cap/Breakout_NEH7100_Cap.kicad_sch (KiCad schematic)
At the start: 41 parts, among them J1 Conn_Breadboard, J2 BAT_EXTRA, SW1 Test, U1 NEH7100

Commit message: Updated BOMs
No PCB changes, just adding Part Number attributes and exporting a table.

Does sneak in a corrected XTAL footprint, but it's not actually applied yet.
Parts:
- CDC1, CFLY4, CIN1, CMPPT1: Part Number (none) -> GRM155R61A104KA01J
- CFLY1, CFLY2: Part Number (none) -> GRM153R61A105ME95D
- CFLY3: Part Number (none) -> GRM155R61A474KE15D
- COUT1: Part Number (none) -> GRM188R60J476ME15D
- CSTR1: Digikey Part Number 1276-1028-1-ND -> (none); Part Number (none) -> GRM188R60J476ME15D
- C_BAT1: Digikey Part Number 490-GRM31CR61A107MEA8LCT-ND -> (none); Part Number (none) -> GRM31CR61A107MEA8L
- C_BAT2, C_BAT3, C_BAT4, C_BAT5: Part Number (none) -> GRM31CR61A107MEA8L
- D3: Part Number (none) -> 150060VS75000
- R1: value 4.7k -> 1k; Digikey Part Number 13-RC0603FR-101KLCT-ND -> (none); Part Number (none) -> RC0603FR-101KL
- R2, R3: Part Number (none) -> RC0603FR-0710KL
- SW1: Digikey Part Number 4809-SKRKAHE020CT-ND -> (none)
- TP1, TP2, TP3, TP6: now left out of the parts list
- U1: Part Number (none) -> NEH7100BUHP
