File: HW/BL54L15μ_DevKit/BL54L15μ_DevKit.kicad_pcb (KiCad board)
At the start: 4 copper layers, 25.4 x 43.2 mm, 42 parts, among them IC1 nrf54L 453-00223R, J1 Conn_Qwiic_1, J2 USB_C_Receptacle, J3 Conn_01x12_Pin, J4 Conn_01x12_Pin, J5 Conn_01x02, J6 Conn_01x02, J7 Conn_01x02, J8 Conn_Qwiic_2, SW1 Button0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

Commit message: BL54L15μ nPM1304 DevKit 2026v2 - Fix LFXO crystal outline to be large enough for actual crystal - Add UART RX/TX via USB-C connector - Reduce to two I2C buses, with one directly VDD powered - Add more test points - Add silkscreen outline to Ezurio 453-00223R footprint for DFM - Various cleanups, delete unused footprints
Parts:
- removed D1: PWRLED, LED_SMD:LED_0603_1608Metric
- removed R1: 2kΩ, Resistor_SMD:R_0402_1005Metric
- added JP1: UART_TXD, Jumper:SolderJumper-2_P1.3mm_Bridged_RoundedPad1.0x1.5mm, B.Cu at (65.6, 107.5)
- added JP2: UART_RXD, Jumper:SolderJumper-2_P1.3mm_Bridged_RoundedPad1.0x1.5mm, B.Cu at (68.1, 107.5)
- added TP3: ~{RESET}, TestPoint:TestPoint_Pad_D1.0mm, B.Cu at (51.8, 80.7)
- added TP4: P1.07, TestPoint:TestPoint_Pad_D1.0mm, B.Cu at (51.4, 90.7)
- added TP5: P1.08, TestPoint:TestPoint_Pad_D1.0mm, B.Cu at (51.5, 88.3)
- C3: value 10uF -> 10μF
- U1: value nPM1300-QEXX -> NPM1304-QEAA
- X1: footprint Crystal:Crystal_SMD_2012-2Pin_2.0x1.2mm -> CM7V_T1A_LOW_ESR_32_768KHZ_9PF_20_TA_QC:XTAL_CM7V-T1A-LOW-ESR-32.768KHZ-9PF-20-TA-QC
- moved C3 0.28 mm to (56.4, 86.0)
Connections:
- IC1 pad 29: /SCL2 -> /P0.04/CLK
- IC1 pad 30: /SDA2 -> /P0.02
- J1 pad 2: LSOUT1 -> /nVDD
- J1 pad 3: /SDA1 -> /SDA0
- J1 pad 4: /SCL1 -> /SCL0
- J2 pad B10: unconnected-(J2-RX1--PadB10) -> /UART_TXD
- J2 pad B11: unconnected-(J2-RX1+-PadB11) -> /UART_RXD
- J8 pad 3: /SDA2 -> /SDA1
- J8 pad 4: /SCL2 -> /SCL1
Routing:
- net /P0.02: track 0.00 -> 35.9 mm, vias 0 -> 3
- net /P0.04/CLK: track 0.00 -> 35.7 mm, vias 0 -> 3
- net /VBUSOUT: track 39.1 -> 12.8 mm, vias 2 -> 0
- net /UART_RXD: track 0.00 -> 17.7 mm, vias 0 -> 1
- net /SCL2: track 17.0 -> 0.00 mm, vias 2 -> 0
- net /SDA2: track 16.7 -> 0.00 mm, vias 2 -> 0
- net LSOUT1: track 27.5 -> 11.6 mm, vias 4 -> 0
- net /UART_TXD: track 0.00 -> 14.1 mm, vias 0 -> 1
- net /SDA0: track 31.3 -> 38.2 mm, vias 4 -> 5
- net /SCL0: track 28.4 -> 34.1 mm
- net /SDA1: track 14.7 -> 9.29 mm
- net /nVDD: track 49.5 -> 53.2 mm
- net /SCL1: track 13.5 -> 10.1 mm
- net /P1.14: track 27.1 -> 29.7 mm
- net /P1.13: track 30.4 -> 32.9 mm
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Other:
- board text added: "1.08"
- board text added: "I²C STEMMA QT Load switched"
- board text added: "|1.05|LS2|"
- board text added: "|1.07|VDD|"
- board text removed: "0.04"
- board text removed: "Battery 3.5- 4.45 V Li-ion/Li-poly/LiFePO_{4}"
- board text removed: "I²C STEMMA QT's Load switched"
- board text removed: "NTC Thermistor JST PH 2mm pitch"
- board text removed: "USB"
- board text removed: "|0.02|LS2|"
- board text removed: "|1.05|LS1|"
