File: HW/BL54L15μ_DevKit/BL54L15μ_DevKit.kicad_sch (KiCad schematic)
At the start: 42 parts, among them IC1 nrf54L 453-00223R, J1 Conn_Qwiic_1, J2 USB_C_Receptacle, J3 Conn_01x12_Pin, J4 Conn_01x12_Pin, J5 Conn_01x02, J6 Conn_01x02, J7 Conn_01x02, J8 Conn_Qwiic_2, SW1 Button0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

Commit message: Updated BOMs
No PCB changes, just adding Part Number attributes and exporting a table.

Does sneak in a corrected XTAL footprint, but it's not actually applied yet.
Parts:
- C1, C5: Part Number (none) -> CL05A105KA5NQNC
- C10, C11, C2, C4, C7: Digikey Part Number 1276-1869-1-ND -> (none); Part Number (none) -> CL10A106KP8NNNC
- C12: Part Number (none) -> CL05B103KB5NNNC
- C3: Part Number (none) -> CL10A106KP8NNNC
- C6: Part Number (none) -> CL05A225KP5NSNC
- C8, C9: Digikey Part Number 1276-1182-1-ND -> (none); Part Number (none) -> CL10A105KP8NNNC
- D1: Part Number (none) -> 150060GS75000
- D2: Part Number (none) -> 150060SS75000
- D3: Part Number (none) -> 150352M173300
- IC1: Manufacturer_Part_Number 453-00223R -> (none); Part Number (none) -> 453-00223R
- J1, J8: Part Number (none) -> BM04B-SRSS-TB
- J2: Part Number (none) -> USB4056-03-A
- J6, J7: Part Number (none) -> B2B-PH-K-S
- L1, L2: Part Number (none) -> CIGT201610EH2R2MNE
- R1: Part Number (none) -> RC0402FR-132KL
- R2: Part Number (none) -> RC0603JR-07330KL
- R3: Digikey Part Number RC0603FR-0747KL -> (none); Part Number (none) -> RC0603FR-0747KL
- R4: Digikey Part Number 13-RC0402FR-132KLCT-ND -> (none); Part Number (none) -> RC0603FR-07100RL
- TP1, TP2: now left out of the parts list
- U1: value nPM1300-QEXX -> NPM1304-QEAA; Part Number (none) -> NPM1304-QEAA-R7
- X1: Digikey Part Number 2195-CM7VT1ALOWESR32.768KHZ9PF20TAQCCT-ND -> (none); Part Number (none) -> CM7V-T1A-LOW-ESR-32.768KHZ-9PF-20-TA-QC

Commit message: BL54L15μ nPM1304 DevKit 2026v2 - Fix LFXO crystal outline to be large enough for actual crystal - Add UART RX/TX via USB-C connector - Reduce to two I2C buses, with one directly VDD powered - Add more test points - Add silkscreen outline to Ezurio 453-00223R footprint for DFM - Various cleanups, delete unused footprints
Parts:
- removed D1: PWRLED, LED_SMD:LED_0603_1608Metric, symbol Device:LED
- removed R1: 2kΩ, Resistor_SMD:R_0402_1005Metric, symbol Device:R
- added JP1: UART_TXD, Jumper:SolderJumper-2_P1.3mm_Bridged_RoundedPad1.0x1.5mm, symbol Jumper:SolderJumper_2_Bridged
- added JP2: UART_RXD, Jumper:SolderJumper-2_P1.3mm_Bridged_RoundedPad1.0x1.5mm, symbol Jumper:SolderJumper_2_Bridged
- added TP3: ~{RESET}, TestPoint:TestPoint_Pad_D1.0mm, symbol Connector:TestPoint
- added TP4: P1.07, TestPoint:TestPoint_Pad_D1.0mm, symbol Connector:TestPoint
- added TP5: P1.08, TestPoint:TestPoint_Pad_D1.0mm, symbol Connector:TestPoint
- C3: value 10uF -> 10μF
- X1: footprint Crystal:Crystal_SMD_2012-2Pin_2.0x1.2mm -> CM7V_T1A_LOW_ESR_32_768KHZ_9PF_20_TA_QC:XTAL_CM7V-T1A-LOW-ESR-32.768KHZ-9PF-20-TA-QC
Connections:
- net LSOUT1: no longer J1.2
- net SCL0: now also J1.4, TP5.1
- net SCL1: now also J8.4; no longer J1.4
- net SDA0: now also J1.3, TP4.1
- net SDA1: now also J8.3; no longer J1.3
- net nVDD: now also J1.2
- net ~{RESET}: now also TP3.1
- net UART_TXD: now reaches J2.B10 (RX1-)
- net UART_TXD: now also JP1.1 (A)
- net UART_RXD: now reaches J2.B11 (RX1+)
- net UART_RXD: now also JP2.1 (A)
- net SCL2 renamed P0.04/CLK
- net P0.04/CLK: now also JP1.2 (B); no longer J8.4
- net SDA2 renamed P0.02
- net P0.02: now also JP2.2 (B); no longer J8.3
- no-connect marks 17 -> 15
Other:
- note added: "BL54L15μ"
- note added: "LED"
- note removed: "BL54L15μ (nrf54L15 module)"
- note removed: "LEDs"
- moved on the sheet: D2, R4, SW1, SW2, TP1, TP2

Commit message: Tweaks
Parts:
- R2: value 250-500 kΩ -> 150kΩ; Digikey Part Number 311-330KGRCT-ND -> (none); Part Number RC0603JR-07330KL -> RC0603FR-07150KL
- R3: value 47 kΩ -> 47kΩ
Changed lines of the file:
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@@
 			)
 		)
-		(property "Value" "47 kΩ"
+		(property "Value" "47kΩ"
 			(at 26.67 176.5299 0)
 			(effects
@@
 			)
 		)
-		(property "Value" "250-500 kΩ"
+		(property "Value" "150kΩ"
 			(at 36.83 181.6099 0)
 			(effects
@@
 			)
 		)
-		(property "Digikey Part Number" "311-330KGRCT-ND"
+		(property "Part Number" "RC0603FR-07150KL"
 			(at 34.29 180.34 0)
 			(effects
-				(font
-					(size 1.27 1.27)
-				)
-				(hide yes)
-			)
-		)
-		(property "Part Number" "RC0603JR-07330KL"
-			(at 34.29 180.34 0)
-			(effects
