File: HW/BL54L15μ_Solar_DevKit/BL54L15μ_Solar_DevKit.kicad_pcb (KiCad board)
At the start: 4 copper layers, 20.3 x 30.5 mm, 35 parts, among them IC1 nrf54L 453-00223R, J1 Conn_Qwiic_1, J2 USB_C_Receptacle, J3 Conn_01x12_Pin, J4 Conn_01x12_Pin, SW1 Button0, U1 NEH7100, X1 32.768 kHz

Commit message: Layout WIP
Parts:
- removed CBAT1: 47u, Capacitor_SMD:C_0603_1608Metric
- removed the D2 at (50.5, 102.5)
- removed the J1 at (54.9, 87.7)
- removed the J1 at (64.5, 87.6)
- removed REF**: JST_PH_S2B-PH-K_1x02_P2.00mm_Horizontal, Connector_JST:JST_PH_S2B-PH-K_1x02_P2.00mm_Horizontal
- removed REF**: JST_PH_B2B-PH-K_1x02_P2.00mm_Vertical, Connector_JST:JST_PH_B2B-PH-K_1x02_P2.00mm_Vertical
- removed REF**: JST_SH_SM04B-SRSS-TB_1x04-1MP_P1.00mm_Horizontal, Connector_JST:JST_SH_SM04B-SRSS-TB_1x04-1MP_P1.00mm_Horizontal
- added J5: Conn_01x02, Connector_JST:JST_PH_B2B-PH-K_1x02_P2.00mm_Vertical, F.Cu at (63.9, 88.5)
- J3, J4: footprint Connector_PinHeader_2.54mm:PinHeader_1x08_P2.54mm_Vertical -> Connector_PinHeader_2.54mm_SilkFree:PinHeader_1x12_P2.54mm_Vertical
- moved J1 50.8 mm to (55.0, 87.6), turned to 90 degrees
- moved J2 3.14 mm to (59.7, 103.9)
- moved D2 2.35 mm to (65.3, 77.2)
- moved R4 1.37 mm to (65.3, 80.4), turned to 90 degrees
- moved U1 0.12 mm to (59.7, 93.6)
- moved CFLY2 0.09 mm to (58.6, 89.9)
- moved X1 0.05 mm to (59.7, 85.2)
Connections:
- COUT1 pad 1: VOUT -> VDD
- IC1 pad 5: /nVDD -> VDD
- J2 pad A4: VBUS -> +5V
- J2 pad A8: /nVDD -> VDD
- J2 pad A9: VBUS -> +5V
- J2 pad B10: unconnected-(J2-RX1--PadB10) -> /UART_TXD
- J2 pad B11: unconnected-(J2-RX1+-PadB11) -> /UART_RXD
- J2 pad B4: VBUS -> +5V
- J2 pad B9: VBUS -> +5V
- J3 pad 7: (no net) -> /P1.14
- J3 pad 8: (no net) -> /P1.13
- J4 pad 4: GND -> unconnected-(J4-Pin_4-Pad4)
- J4 pad 5: VOUT1 -> unconnected-(J4-Pin_5-Pad5)
- J4 pad 6: VOUT2 -> unconnected-(J4-Pin_6-Pad6)
- J4 pad 7: /LSOUT2 -> unconnected-(J4-Pin_7-Pad7)
- J4 pad 8: /LSOUT1 -> unconnected-(J4-Pin_8-Pad8)
- U1 pad 13: VOUT -> VDD
Routing:
- net GND: track 126.4 -> 54.6 mm, vias 55 -> 40
- net /nVDD: track 18.5 -> 0.00 mm
- net /GPIO4: track 12.3 -> 0.00 mm
- net VOUT1: track 10.8 -> 0.00 mm
- net /SCL0: track 28.4 -> 18.2 mm
- net /P2.05: track 12.4 -> 3.85 mm
- net VBUS: track 7.60 -> 0.00 mm, vias 1 -> 0
- net /CMPPT: track 6.67 -> 0.00 mm
- net /SDA0: track 27.7 -> 21.1 mm, vias 4 -> 3
- net /P1.14: track 22.1 -> 15.5 mm
- net /P1.15: track 23.3 -> 16.8 mm
- net /P2.01/CLK: track 12.1 -> 6.46 mm, vias 3 -> 2
- net /P2.00: track 11.6 -> 6.10 mm, vias 0 -> 1
- net /SWDIO: track 47.0 -> 42.0 mm, vias 2 -> 1
- net /P2.04: track 8.95 -> 5.55 mm
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- removed copper zone on F.Cu, net VSYS

Commit message: Almost complete schematic plus basic routing
Parts:
- J3, J4: footprint Connector_PinHeader_2.54mm_SilkFree:PinHeader_1x12_P2.54mm_Vertical -> Connector_PinHeader_2.54mm_SilkFree:PinHeader_1x11_P2.54mm_Vertical
- moved CIN1 2.30 mm to (64.6, 92.1), turned to -90 degrees
- moved CSTR1 1.47 mm to (64.6, 94.1)
- moved CDC1 0.30 mm to (54.4, 92.6)
- moved CMPPT1 0.29 mm to (54.4, 95.2)
- moved CFLY3 0.19 mm to (55.9, 92.6)
- moved CFLY4 0.15 mm to (55.9, 95.1)
Connections:
- COUT1 pad 1: VDD -> VLDO
- IC1 pad 3: /SCL0 -> /SCL
- IC1 pad 8: /SDA0 -> /SDA
- J1 pad 2: unconnected-(J1-Pad2) -> VDD
- J1 pad 3: /SDA1 -> /SDA
- J1 pad 4: /SCL1 -> /SCL
- J3 pad 11: unconnected-(J3-Pin_11-Pad11) -> GND
- J4 pad 10: /VBUS -> /VBAT
- J4 pad 11: /VBAT -> GND
- J4 pad 6: unconnected-(J4-Pin_6-Pad6) -> /VOUT_EN
- J4 pad 7: unconnected-(J4-Pin_7-Pad7) -> /VBAT_OK
- J4 pad 8: unconnected-(J4-Pin_8-Pad8) -> /VIN
- J4 pad 9: unconnected-(J4-Pin_9-Pad9) -> /VBUS
- JP3 pad 1: GND -> /VSTOR
- JP3 pad 3: /VSTOR -> GND
- JP4 pad 1: GND -> /VSTOR
- JP4 pad 3: /VSTOR -> GND
- JP6 pad 1: GND -> /VSTOR
- JP6 pad 3: /VSTOR -> GND
- JP7 pad 1: GND -> /VSTOR
- JP7 pad 3: /VSTOR -> GND
- U1 pad 13: VDD -> VLDO
Routing:
- net GND: track 54.6 -> 4.12 mm, vias 40 -> 22
- net /SDA0: track 21.1 -> 0.00 mm, vias 3 -> 0
- net /SWDCLK: track 42.6 -> 24.3 mm
- net /SCL0: track 18.2 -> 0.00 mm, vias 2 -> 0
- net /SWDIO: track 42.0 -> 25.0 mm
- net /~{RESET}: track 38.3 -> 22.6 mm
- net /SCL2: track 15.6 -> 5.94 mm
- net /SDA: track 0.00 -> 9.13 mm, vias 0 -> 1
- net /SDA2: track 15.5 -> 6.93 mm
- net (no net): track 7.82 -> 0.21 mm
- net /P1.02/NFC1: track 14.2 -> 8.20 mm
- net /VIN: track 0.00 -> 5.63 mm
- net /VSTOR: track 0.00 -> 5.19 mm
- net /SCL: track 0.00 -> 4.56 mm
- net /CMPPT: track 0.00 -> 4.14 mm
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
Commit message: WIP
Parts:
- added CBAT1: 47u, Capacitor_SMD:C_0603_1608Metric, F.Cu at (64.9, 93.6)
- added J2: USB_C_Receptacle, USB4056_03_A:GCT_USB4056-03-A_REVA2, F.Cu at (57.0, 126.8)
- added J5: Batt_JST-PH-B2B, Connector_JST:JST_PH_B2B-PH-K_1x02_P2.00mm_Vertical, F.Cu at (90.7, 116.0)
- added R1: 5.1kΩ, Resistor_SMD:R_0603_1608Metric, F.Cu at (53.4, 103.1)
- added R2: 5.1kΩ, Resistor_SMD:R_0603_1608Metric, F.Cu at (65.8, 103.2)
- added REF**: JST_ZH_B2B-ZR_1x02_P1.50mm_Vertical, Connector_JST:JST_ZH_B2B-ZR_1x02_P1.50mm_Vertical, F.Cu at (64.3, 88.1)
- added REF**: PinHeader_1x02_P2.54mm_Vertical, Connector_PinHeader_2.54mm:PinHeader_1x02_P2.54mm_Vertical, F.Cu at (53.4, 80.0)
- added REF**: JST_PH_S2B-PH-K_1x02_P2.00mm_Horizontal, Connector_JST:JST_PH_S2B-PH-K_1x02_P2.00mm_Horizontal, F.Cu at (64.6, 122.9)
- J5: value Conn_01x02 -> Batt_JST-PH-B2B
- JP8: value OUTEN_BATOK -> LDOEN_BATOK
- moved J5 26.8 mm to (84.0, 106.3)
- moved SW1 11.4 mm to (65.5, 81.1)
- moved COUT1 9.03 mm to (64.9, 95.5)
- moved CIN1 4.61 mm to (61.0, 89.4), turned to 90 degrees
- moved R4 3.70 mm to (64.6, 76.8), turned to -90 degrees
- moved JP9 2.75 mm to (97.7, 66.6)
- moved CSTR1 2.43 mm to (64.9, 91.7)
- moved CFLY1 1.21 mm to (59.7, 89.4), turned to -90 degrees
- moved D2 0.83 mm to (66.0, 76.8)
- moved CFLY2 0.63 mm to (58.4, 89.3), turned to -90 degrees
- moved CDC1 0.13 mm to (54.4, 92.5)
- moved CFLY3 0.13 mm to (55.9, 92.5)
Connections:
- net /GPIO1 renamed /P0.01
- net /GPIO2 renamed /P0.03/CLK
- net /SCL1 renamed /P1.04/AIN0/CLK
- net /SCL2 renamed /P0.04/CLK
- net /SDA1 renamed /P1.05
- net /SDA2 renamed /P0.02
- J3 pad 10: unconnected-(J3-Pin_10-Pad10) -> /VBUS
- J4 pad 10: /VBAT -> /VBAT_OK
- J4 pad 11: GND -> unconnected-(J4-Pin_11-Pad11)
- J4 pad 5: unconnected-(J4-Pin_5-Pad5) -> GND
- J4 pad 6: /VOUT_EN -> /VIN
- J4 pad 7: /VBAT_OK -> /VBAT
- J4 pad 8: /VIN -> VLDO
- J4 pad 9: /VBUS -> /LDO_EN
- JP8 pad 2: /VOUT_EN -> /LDO_EN
- U1 pad 12: /VOUT_EN -> /LDO_EN
Routing:
- net /UART_RXD: track 0.00 -> 33.4 mm, vias 0 -> 2
- net /UART_TXD: track 0.00 -> 32.2 mm, vias 0 -> 2
- net /P0.03/CLK: track 21.5 -> 0.00 mm, vias 1 -> 0
- net /P0.01: track 20.6 -> 0.00 mm, vias 1 -> 0
- net +5V: track 0.00 -> 18.8 mm, vias 0 -> 1
- net /~{RESET}: track 22.6 -> 39.2 mm
- net /P1.14: track 15.5 -> 1.04 mm
- net /P1.13: track 17.3 -> 3.53 mm
- net /P1.15: track 17.0 -> 3.45 mm
- net /P1.05: track 13.0 -> 0.48 mm
- net /VBAT: track 0.00 -> 12.5 mm, vias 0 -> 1
- net /P1.04/AIN0/CLK: track 11.5 -> 0.48 mm
- net /CC1: track 0.00 -> 10.4 mm, vias 0 -> 2
- net /SWDIO: track 25.0 -> 34.1 mm, vias 1 -> 2
- net /SWDCLK: track 24.3 -> 32.8 mm, vias 1 -> 2
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Other:
- board size 20.3 x 30.5 mm -> 20.3 x 53.4 mm
