File: HW/BL54L15μ_Solar_DevKit/BL54L15μ_Solar_DevKit.kicad_sch (KiCad schematic)
At the start: 29 parts, among them IC1 nrf54L 453-00223R, J1 Conn_Qwiic_1, J2 USB_C_Receptacle, J3 Conn_01x12_Pin, J4 Conn_01x12_Pin, SW1 Button0, U1 NEH7100, X1 32.768 kHz

Commit message: Layout WIP
Parts:
- removed C3: 10uF, Capacitor_SMD:C_0603_1608Metric, symbol Device:C
- added J5: Conn_01x02, Connector_JST:JST_PH_B2B-PH-K_1x02_P2.00mm_Vertical, symbol Connector_Generic:Conn_01x02
- J3, J4: footprint Connector_PinHeader_2.54mm_SilkFree:PinHeader_1x12_P2.54mm_Vertical -> Connector_PinHeader_2.54mm_SilkFree:PinHeader_1x11_P2.54mm_Vertical; symbol Connector:Conn_01x12_Pin -> Connector:Conn_01x11_Pin
Connections:
- net VBUSOUT is gone; now on net VBUS: J4.10 (Pin_10)
- net nVDD is gone; now on net VDD: IC1.5 (VDD_NRF), J2.A8 (SBU1)
- net +5V: now also J2.A4 (VBUS), J2.A9 (VBUS), J2.B4 (VBUS), J2.B9 (VBUS)
- net GND: now also J5.1 (Pin_1); no longer J3.12 (Pin_12), J4.12 (Pin_12), J4.4 (Pin_4)
- net VBAT: now also J5.2 (Pin_2)
- net VBUS: no longer J2.A4 (VBUS), J2.A9 (VBUS), J2.B4 (VBUS), J2.B9 (VBUS)
- net UART_TXD: now reaches J2.B10 (RX1-)
- net UART_RXD: now reaches J2.B11 (RX1+)
- net GPIO3: no longer names the net of J3.9 (Pin_9)
- net GPIO4: no longer names the net of J3.10 (Pin_10)
- net LSOUT1: no longer names the net of J4.8 (Pin_8)
- net LSOUT2: no longer names the net of J4.7 (Pin_7)
- net NTC: no longer names the net of J3.11 (Pin_11)
- net VOUT renamed VDD
- net VOUT1: no longer names the net of J4.5 (Pin_5)
- net VOUT2: no longer names the net of J4.6 (Pin_6)
- net VSYS: no longer names the net of J4.9 (Pin_9)
- no-connect marks 18 -> 16
Other:
- note added: "Button"
- note added: "I2C Address: 0x6B Inductorless energy harvesting PMIC 15 μW to 100 mW input with MPTT USB charging up to 200 mA 200 mA LDO, 130 mV dropout Quiescent current 1.5 μA (2.1 with LDO)"
- note added: "I^{2}C Connector"
- note added: "LED"
- note added: "NEH7100"
- note removed: "Buttons"
- note removed: "I2C Address: 0x6B 4 mA to 100 mA USB-C battery charger Two 200 mA buck regulators Two 100 mA load switches / 50mA LDOs"
- note removed: "LEDs"
- note removed: "Qwicc I^{2}C Connectors"
- note removed: "nPM1304 PMIC"
- moved on the sheet: D2, R4, SW1

Commit message: Almost complete schematic plus basic routing
Parts:
- added JP1: SolderJumper_2_Bridged, symbol Jumper:SolderJumper_2_Bridged
- added R1, R2: 5.1kΩ, symbol Device:R
Connections:
- net GPIO1 is gone; now on net UART_TXD: IC1.35 (P0.01)
- net GPIO2 is gone; now on net UART_RXD: IC1.33 (P0.03/CLK)
- net SCL0 is gone; now on net SCL: IC1.3 (P1.08/EXTREF/CLK16M/CLK)
- net SDA0 is gone; now on net SDA: IC1.8 (P1.07)
- net +5V: now also R1.2, R2.2
- net CC1: now also R1.1
- net CC2: now also R2.1
- net GND: now also J3.11 (Pin_11), J4.11 (Pin_11), JP3.3 (B), JP4.3 (B), JP6.3 (B), JP7.3 (B); no longer JP3.1 (A), JP4.1 (A), JP6.1 (A), JP7.1 (A)
- net SCL: now also J1.4
- net SCL1: no longer J1.4
- net SDA: now also J1.3
- net SDA1: no longer J1.3
- net VBAT: now also J4.10 (Pin_10); no longer J4.11 (Pin_11)
- net VBAT_OK: now also J4.7 (Pin_7)
- net VBUS: now also J4.9 (Pin_9); no longer J4.10 (Pin_10)
- net VDD: now also J1.2, JP1.2 (B); no longer COUT1.1, U1.13 (VLDO)
- net VIN: now also J4.8 (Pin_8)
- net VOUT_EN: now also J4.6 (Pin_6)
- net VSTOR: now also JP3.1 (A), JP4.1 (A), JP6.1 (A), JP7.1 (A); no longer JP3.3 (B), JP4.3 (B), JP6.3 (B), JP7.3 (B)
- net SCL2: no longer names the net of IC1.29 (P0.04/CLK)
- net SDA2: no longer names the net of IC1.30 (P0.02)
- new net VLDO: COUT1.1, JP1.1 (A), U1.13 (VLDO)
Other:
- note added: "Hard-coded settings Interpreted during power-up Connected to either "0" (GND) or "1" (VSTOR) May be overriden via I²C registers See section 7.3.7 in datasheet Default chosen for LFP/LiFePO4: 11011: OVP=3.5V LVD=2.5V LDO=Pass OCP=150mA Alternate to solder for NMC/etc: 00000: OVP=4.2V LVD=3.5V LDO=3.3V OCP=200mA"
- note added: "I2C Address: 0x3C Inductorless energy harvesting PMIC Battery charger with OVP/LVP 15 μW to 100 mW input with MPTT USB charging up to 200 mA 200 mA LDO, 130 mV dropout Quiescent current 1.5 μA (2.1 with LDO)"
- note removed: "I2C Address: 0x6B Inductorless energy harvesting PMIC 15 μW to 100 mW input with MPTT USB charging up to 200 mA 200 mA LDO, 130 mV dropout Quiescent current 1.5 μA (2.1 with LDO)"
- note removed: "See section 7.3.7 in datasheet for hard-code settings Connected to either "0" (GND) or "1" (VSTOR) Interpreted at the moment of power-up May be overriden via I²C registers after power-up 00000: OVP=4.2V LVD=3.5V LDO=3.3V OCP=200mA 00100: OVP=4.2V LVD=2.2V LDO=1.8V OCP=200mA"
- moved on the sheet: CDC1, CFLY1, CFLY2, CFLY3, CFLY4, CIN1, CMPPT1, COUT1, CSTR1, D2, J1, J2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

Commit message: WIP
Parts:
- added CBAT1: 47u, Capacitor_SMD:C_0603_1608Metric, symbol Device:C
- J5: value Conn_01x02 -> Batt_JST-PH-B2B
- JP8: value OUTEN_BATOK -> LDOEN_BATOK
- R1, R2: footprint (none) -> Resistor_SMD:R_0603_1608Metric
Connections:
- net GND: now also J4.5 (Pin_5), CBAT1.2; no longer J4.11 (Pin_11)
- net UART_RXD: no longer IC1.33 (P0.03/CLK)
- net UART_TXD: no longer IC1.35 (P0.01)
- net VBAT: now also J4.7 (Pin_7), CBAT1.1; no longer J4.10 (Pin_10)
- net VBAT_OK: now also J4.10 (Pin_10); no longer J4.7 (Pin_7)
- net VBUS: now also J3.10 (Pin_10); no longer J4.9 (Pin_9)
- net VDD: no longer JP1.2 (B)
- net VIN: now also J4.6 (Pin_6); no longer J4.8 (Pin_8)
- net VLDO: now also J4.8 (Pin_8), JP1.2 (B)
- net P0.04/CLK: now reaches IC1.29 (P0.04/CLK)
- net P0.02: now reaches IC1.30 (P0.02)
- net SCL1 renamed P1.04/AIN0/CLK
- net SDA1 renamed P1.05
- net VOUT_EN renamed LDO_EN
- net LDO_EN: now also J4.9 (Pin_9); no longer J4.6 (Pin_6)
- new net P0.01: IC1.35 (P0.01)
- new net P0.03/CLK: IC1.33 (P0.03/CLK)
Other:
- moved on the sheet: J5, JP1

Commit message: Tweaks
Parts:
- R1, R2: Part Number (none) -> RC0603FR-075K1L
Changed lines of the file:
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@@
+			)
+		)
+		(property "Part Number" "RC0603FR-075K1L"
+			(at 72.39 24.13 0)
+			(effects
+				(font
+					(size 1.27 1.27)
+				)
+				(hide yes)
 			)
 		)
@@
 			(at 62.23 24.13 0)
 			(effects
+				(font
+					(size 1.27 1.27)
+				)
+				(hide yes)
+			)
+		)
+		(property "Part Number" "RC0603FR-075K1L"
+			(at 62.23 24.13 0)
+			(effects
