File: HW/SWD_USBC_InlineAdapter/SWD_USBC_InlineAdapter.kicad_sch (KiCad schematic)
At the start: 7 parts, among them J1 Conn_ARM_JTAG_SWD_10, J5 USB_C_Receptacle_USB2.0_14P, P1 USB_C_Plug

Commit message: SWD to USB-C adapter 2026r2
Parts:
- removed J5: USB_C_Receptacle_USB2.0_14P, Connector_USB:USB_C_Receptacle_GCT_USB4085, symbol Connector:USB_C_Receptacle_USB2.0_14P
- added D1: RED LED, Diode_SMD:D_0603_1608Metric, symbol Device:LED
- added J2: Conn_01x04, Connector_Molex:Molex_PicoBlade_53261-0471_1x04-1MP_P1.25mm_Horizontal, symbol Connector_Generic:Conn_01x04
- added J3: USB_C_Receptacle, USB4056_03_A:GCT_USB4056-03-A_REVA2, symbol Connector:USB_C_Receptacle
- added R1: 100Ω, Resistor_SMD:R_0603_1608Metric, symbol Device:R
- J1: footprint Connector_PinHeader_1.27mm:PinHeader_2x05_P1.27mm_Vertical -> Connector_PinHeader_1.27mm:PinHeader_2x05_P1.27mm_Vertical_SMD; Manufacturer (none) -> Samtec Inc.; Part Number (none) -> FTSH-105-01-F-DV-K
- P1: symbol USB_C:USB_C_Plug_SWD -> USBC_Connector:USB_C_Plug; Part Number (none) -> USB4155-03-C
- renumbered R6 to R2, R4 to R3, R7 to R4, R8 to R5
Connections:
- net +5V: now also J3.A4 (VBUS), J3.A9 (VBUS), J3.B4 (VBUS), J3.B9 (VBUS)
- net CC1_SRC: now also J3.A5 (CC1)
- net CC2_SRC: now also J3.B5 (CC2)
- net D+: now also J3.A6 (D+), J3.B6 (D+)
- net D-: now also J3.A7 (D-), J3.B7 (D-)
- net GND: now also D1.1 (K), J3.A1 (GND), J3.A12 (GND), J3.B1 (GND), J3.B12 (GND), J3.S1 (SHIELD)
- net UART_TXD: now reaches P1.B10 (RX1-)
- net UART_TXD: now also J2.2 (Pin_2)
- net UART_RXD: now reaches P1.B11 (RX1+)
- net UART_RXD: now also J2.3 (Pin_3)
- net Tgnd renamed tGND
- net tGND: now also J2.4 (Pin_4), R1.1
- net VTref renamed tVDD
- net tVDD: now also J2.1 (Pin_1)
- new net: D1.2 (A), R1.2
- no-connect marks 5 -> 13
Other:
- note added: "Layout 2x05, 1.27mm pitch"
- note added: "Lit only when plug is upside down"
- note added: "Molex PicoBlade 4-pin, 1.25mm pitch"
- note added: "Reversal Indicator"
- note added: "UART Connector"
- note removed: "Layout 2x05, Pitch 1.27mm"
- moved on the sheet: R4, R5

Commit message: SWB to USB adapter bill of materials
Parts:
- J3, P1: Manufacturer (none) -> GCT
- R2: Digikey Part Number RC0603FR-1322KL -> (none); Part Number (none) -> RC0603FR-1322KL
- R3: Digikey Part Number RC0603FR-0710KL -> (none); Part Number (none) -> RC0603FR-0710KL
- R4, R5: Digikey Part Number 311-5.10KHRCT-ND -> (none); Part Number (none) -> RC0603FR-075K1L
Changed lines of the file:
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@@
+			)
+		)
+		(property "Manufacturer" "GCT"
+			(at 241.3 85.09 0)
+			(effects
+				(font
+					(size 1.27 1.27)
+				)
+				(hide yes)
+			)
+		)
+		(property "Digikey Part Number" ""
+			(at 241.3 85.09 0)
+			(effects
+				(font
+					(size 1.27 1.27)
+				)
+				(hide yes)
 			)
 		)
 		(property "Manufacturer_Part_Number" ""
-			(at 241.3 85.09 90)
+			(at 241.3 85.09 0)
 			(effects
 				(font
@@
 			)
 		)
+		(property "Manufacturer" "GCT"
+			(at 39.37 73.66 0)
+			(effects
+				(font
+					(size 1.27 1.27)
+				)
+				(hide yes)
+			)
+		)
+		(property "Digikey Part Number" ""
+			(at 39.37 73.66 0)
+			(effects
+				(font
+					(size 1.27 1.27)
+				)
+				(hide yes)
+			)
+		)
+		(property "Manufacturer_Part_Number" ""
+			(at 39.37 73.66 0)
+			(effects
+				(font
+					(size 1.27 1.27)
+				)
+				(hide yes)
+			)
+		)
 		(pin "A7"
 		)
@@
 			)
 		)
-		(property "Digikey Part Number" "RC0603FR-0710KL"
+		(property "Part Number" "RC0603FR-0710KL"
+			(at 63.5 49.53 0)
+			(effects
+				(font
+					(size 1.27 1.27)
+				)
+				(hide yes)
+			)
+		)
+		(property "Digikey Part Number" ""
+			(at 63.5 49.53 0)
+			(effects
+				(font
+					(size 1.27 1.27)
+				)
+				(hide yes)
+			)
+		)
+		(property "Manufacturer_Part_Number" ""
 			(at 63.5 49.53 0)
 			(effects
@@
 			)
 		)
+		(property "Digikey Part Number" ""
+			(at 143.51 119.38 0)
+			(effects
+				(font
+					(size 1.27 1.27)
+				)
+				(hide yes)
+			)
+		)
+		(property "Manufacturer_Part_Number" ""
+			(at 143.51 119.38 0)
+			(effects
+				(font
+					(size 1.27 1.27)
+				)
+				(hide yes)
+			)
+		)
 		(pin "4"
 		)
@@
 			)
 		)
-		(property "Digikey Part Number" "311-5.10KHRCT-ND"
+		(property "Part Number" "RC0603FR-075K1L"
+			(at 203.2 68.58 0)
+			(effects
+				(font
+					(size 1.27 1.27)
+				)
+				(hide yes)
+			)
+		)
+		(property "Digikey Part Number" ""
+			(at 203.2 68.58 0)
+			(effects
+				(font
+					(size 1.27 1.27)
+				)
+				(hide yes)
+			)
+		)
+		(property "Manufacturer_Part_Number" ""
 			(at 203.2 68.58 0)
 			(effects
@@
 			)
 		)
-		(property "Digikey Part Number" "RC0603FR-1322KL"
+		(property "Part Number" "RC0603FR-1322KL"
+			(at 80.01 52.07 0)
+			(effects
+				(font
+					(size 1.27 1.27)
+				)
+				(hide yes)
+			)
+		)
+		(property "Digikey Part Number" ""
+			(at 80.01 52.07 0)
+			(effects
+				(font
+					(size 1.27 1.27)
+				)
+				(hide yes)
+			)
+		)
+		(property "Manufacturer_Part_Number" ""
 			(at 80.01 52.07 0)
 			(effects
@@
 			)
 		)
+		(property "Digikey Part Number" ""
+			(at 139.7 58.42 0)
+			(effects
+				(font
+					(size 1.27 1.27)
+				)
+				(hide yes)
+			)
+		)
+		(property "Manufacturer_Part_Number" ""
+			(at 139.7 58.42 0)
+			(effects
+				(font
+					(size 1.27 1.27)
+				)
+				(hide yes)
+			)
+		)
 		(pin "5"
 		)
@@
 			)
 		)
-		(property "Digikey Part Number" "311-5.10KHRCT-ND"
+		(property "Part Number" "RC0603FR-075K1L"
+			(at 213.36 71.12 0)
+			(effects
+				(font
+					(size 1.27 1.27)
+				)
+				(hide yes)
+			)
+		)
+		(property "Digikey Part Number" ""
+			(at 213.36 71.12 0)
+			(effects
+				(font
+					(size 1.27 1.27)
+				)
+				(hide yes)
+			)
+		)
+		(property "Manufacturer_Part_Number" ""
 			(at 213.36 71.12 0)
 			(effects
@@
 			)
 		)
+		(property "Digikey Part Number" ""
+			(at 78.74 180.34 90)
+			(effects
+				(font
+					(size 1.27 1.27)
+				)
+				(hide yes)
+			)
+		)
+		(property "Manufacturer_Part_Number" ""
+			(at 78.74 180.34 90)
+			(effects
+				(font
+					(size 1.27 1.27)
+				)
+				(hide yes)
+			)
+		)
 		(pin "2"
 		)
@@
 			(at 78.74 172.72 0)
 			(effects
+				(font
+					(size 1.27 1.27)
+				)
+				(hide yes)
+			)
+		)
+		(property "Digikey Part Number" ""
+			(at 78.74 172.72 0)
+			(effects
+				(font
+					(size 1.27 1.27)
+				)
+				(hide yes)
+			)
+		)
+		(property "Manufacturer_Part_Number" ""
+			(at 78.74 172.72 0)
+			(effects
