File: HW/BL54L15μ_AirHub/BL54L15μ_AirHub.kicad_pcb (KiCad board)
At the start: 2 copper layers, 33 x 33 mm, 11 parts, among them IC1 nrf54L 453-00223R, J3 USB_C_Receptacle, U2 SHT4x, U4 SCD40-D-R2, U5 BME688, X1 32.768 kHz

Commit message: WIP
Parts:
- removed JP1: UART_TXD, Jumper:SolderJumper-2_P1.3mm_Bridged_RoundedPad1.0x1.5mm
- removed JP2: UART_RXD, Jumper:SolderJumper-2_P1.3mm_Bridged_RoundedPad1.0x1.5mm
- added C10: 100nF, Capacitor_SMD:C_0402_1005Metric, F.Cu at (59.9, 95.8)
- added C8: 100nF, Capacitor_SMD:C_0402_1005Metric, F.Cu at (59.9, 93.8)
- added D1: PWRLED, LED_SMD:LED_0603_1608Metric, F.Cu at (63.3, 94.1)
- added R1: 100Ω, Resistor_SMD:R_0603_1608Metric, F.Cu at (63.3, 96.7)
- added TP1: VDD, TestPoint:TestPoint_Pad_D1.0mm, F.Cu at (50.8, 85.1)
- added TP10: PG/RESET, TestPoint:TestPoint_Pad_D1.0mm, F.Cu at (53.9, 97.3)
- added TP11: SYSGDEN, TestPoint:TestPoint_Pad_D1.0mm, F.Cu at (56.9, 85.1)
- added TP12: LED0, TestPoint:TestPoint_Pad_D1.0mm, F.Cu at (56.9, 88.1)
- added TP13: VDDSW, TestPoint:TestPoint_Pad_D1.0mm, F.Cu at (56.9, 91.2)
- added TP2: GND, TestPoint:TestPoint_Pad_1.0x1.0mm, F.Cu at (50.8, 88.1)
- added TP3: GPIO0/P0.01, TestPoint:TestPoint_Pad_D1.0mm, F.Cu at (50.8, 91.2)
- added TP4: GPIO1, TestPoint:TestPoint_Pad_D1.0mm, F.Cu at (50.8, 94.2)
- added TP5: SDA0/P1.14, TestPoint:TestPoint_Pad_D1.0mm, F.Cu at (50.8, 97.3)
- added TP6: SCL0/P1.04, TestPoint:TestPoint_Pad_D1.0mm, F.Cu at (53.9, 85.1)
- added TP7: SDA1/P1.06, TestPoint:TestPoint_Pad_D1.0mm, F.Cu at (53.9, 88.1)
- added TP8: SCL1/P1.08, TestPoint:TestPoint_Pad_D1.0mm, F.Cu at (53.9, 91.2)
- added TP9: SHPHLD, TestPoint:TestPoint_Pad_D1.0mm, F.Cu at (53.9, 94.2)
- added U1: USBLC6-2SC6, Package_TO_SOT_SMD:SOT-23-6, F.Cu at (61.0, 86.0)
- added U6: AP2112K-3.3, Package_TO_SOT_SMD:SOT-23-5, F.Cu at (61.0, 90.6)
- U4: value SCD40-D-R2 -> SCD4X
- moved U4 34.4 mm to (130.5, 76.2)
- moved C7 26.7 mm to (91.6, 81.8), turned to -90 degrees
- moved U2 21.1 mm to (94.4, 81.3), turned to -90 degrees
- moved IC1 19.1 mm to (105.4, 111.2), turned to -90 degrees
- moved C3 10.9 mm to (109.1, 101.0), turned to 0 degrees
- moved X1 6.05 mm to (105.1, 101.0), turned to 180 degrees
Connections:
- C9 pad 1: VDDSW -> VDD
- IC1 pad 42: /SWO -> unconnected-(IC1-P2.07-Pad42)
- J3 pad A2: /SWDIO -> Net-(J3-TX1+)
- J3 pad A3: /SWDCLK -> Net-(J3-TX1-)
- J3 pad A8: /nVDD -> VDD
- J3 pad B10: /UART_TXD -> unconnected-(J3-RX1--PadB10)
- J3 pad B11: /UART_RXD -> unconnected-(J3-RX1+-PadB11)
- J3 pad B3: /SWO -> unconnected-(J3-TX2--PadB3)
- U2 pad 1: /SDA0 -> /SDA
- U2 pad 2: /SCL0 -> /SCL
- U4 pad 19: VDDSW -> VDD
- U4 pad 7: VDDSW -> VDD
- U5 pad 2: VDDSW -> VDD
- U5 pad 3: /SDA1 -> /SDA
- U5 pad 4: /SCL1 -> /SCL
- U5 pad 6: VDDSW -> VDD
- U5 pad 8: VDDSW -> VDD
Routing:
- net VDDSW: track 19.6 -> 0.00 mm
- net VDD: track 11.3 -> 30.9 mm
- net /SDA: track 0.00 -> 18.6 mm
- net /SCL: track 0.00 -> 17.3 mm
- net /SDA0: track 11.6 -> 0.00 mm
- net /SCL0: track 9.92 -> 0.00 mm
- net /SWO: track 7.99 -> 0.00 mm, vias 2 -> 0
- net unconnected-(IC1-P2.07-Pad42): track 0.00 -> 7.99 mm, vias 0 -> 2
- net /SCL1: track 9.73 -> 2.37 mm
- net /SDA1: track 9.00 -> 2.05 mm
Other:
- outline, holes or cut-outs redrawn
