File: HW/BL54L15μ_AirHub/BL54L15μ_AirHub.kicad_sch (KiCad schematic)
At the start: 27 parts, among them IC1 nrf54L 453-00223R, J3 USB_C_Receptacle, U2 SHT4x, U4 SCD4X, U5 BME688, X1 32.768 kHz

Commit message: WIP
Parts:
- removed JP1: UART_TXD, Jumper:SolderJumper-2_P1.3mm_Bridged_RoundedPad1.0x1.5mm, symbol Jumper:SolderJumper_2_Bridged
- removed JP2: UART_RXD, Jumper:SolderJumper-2_P1.3mm_Bridged_RoundedPad1.0x1.5mm, symbol Jumper:SolderJumper_2_Bridged
- added C10: 100nF, Capacitor_SMD:C_0402_1005Metric, symbol Device:C
- added C4: 4.7µF, symbol Device:C
- added C5, C6: 10µF, symbol Device:C
- added R2, R3: 5.1kΩ, symbol Device:R
- added U1: USBLC6-2SC6, Package_TO_SOT_SMD:SOT-23-6, symbol Power_Protection:USBLC6-2SC6
- added U6: AP2112K-3.3, Package_TO_SOT_SMD:SOT-23-5, symbol Regulator_Linear:AP2112K-3.3
- C3: Manufacturer (none) -> Samsung Electro-Mechanics; Part Number CL10A106KP8NNNC -> CL10A106MA8NRNC
Connections:
- net nVDD is gone; now on net VDD: J3.A8 (SBU1)
- net CC1: now also R2.1
- net CC2: now also R3.1
- net GND: now also C10.2, C4.2, C5.2, C6.2, R2.2, R3.2, U1.2 (GND), U6.2 (GND)
- net SCL: now also U2.2 (SCL), U5.4 (SCK)
- net SCL0: no longer U2.2 (SCL)
- net SCL1: no longer U5.4 (SCK)
- net SDA: now also U2.1 (SDA), U5.3 (SDI)
- net SDA0: no longer U2.1 (SDA)
- net SDA1: no longer U5.3 (SDI)
- net SWDCLK: now also U1.6 (I/O1); no longer J3.A3 (TX1-)
- net SWDIO: now also U1.4 (I/O2); no longer J3.A2 (TX1+)
- net VBUS: now also C4.1, U1.5 (VBUS), U6.1 (VIN), U6.3 (EN)
- net VDD: now also C8.1, C9.1, U4.19 (VDD), U4.7 (VDD), U5.2 (CSB), U5.6 (VDDIO), U5.8 (VDD), C10.1, C5.1, C6.1, U6.5 (VOUT)
- net VDDSW: no longer C8.1, C9.1, U4.19 (VDD), U4.7 (VDD), U5.2 (CSB), U5.6 (VDDIO), U5.8 (VDD)
- net SWO: no longer names the net of J3.B3 (TX2-)
- net SWO: no longer IC1.42 (P2.07)
- net UART_RXD: no longer names the net of J3.B11 (RX1+)
- net UART_TXD: no longer names the net of J3.B10 (RX1-)
- new net: J3.A2 (TX1+), U1.3 (I/O2)
- new net: J3.A3 (TX1-), U1.1 (I/O1)
- no-connect marks 28 -> 31
Other:
- note added: "CO₂ SCD4X"
- note added: "I2C Address: 0x62 VDD: 2.4 - 5.5 V peak 205 mA @ 3.3 V, avg 15 mA ripple of less than 30 mV p-p SCD43 CO2 Accuracy: ±(30 ppm + 3%) %RH Accuracy: ±6 in 15 - 35 °C, 20 - 65 %RH °C Accuracy: ± 0.8 in 15 - 35 °C after offsetting"
- note added: "I2C Address: 0x76 VDD: 1.71 V - 3.6 V 0.29 μA idle, 714 μA typ pressure, 12 mA typ gas %RH Accuracy: ±3 °C Accuracy: ± 0.5 in 0 - 65 °C"
- note added: "USB-C Receptacle and Power"
- note removed: "?"
- note removed: "CO₂ SCD5X"
- note removed: "I2C Address: 0x76 VDD: 1.71 V - 3.6 V 0.29 μA idle, 714 μA typ pressure, 12 mA typ gas"
- note removed: "USB-C Receptacle"
- moved on the sheet: C7, C8, C9, D1, J3, R1, U2, U4, U5
